File: AudioCodec.sch (KiCad schematic (older format))
At the start: 44 parts, among them CN1 IO20, CN12 CONN_02X03, J1 SJ-43514-SMT, P1 CONN_01X02, P2 CONN_01X04, P3 CONN_01X04, Q1 2N7002, Q2 2N7002, U1 TPS730, U2 AK4951AEN

Commit message: Add files via upload
Parts:
- added FB7: FB, HERMESLITE:C_0603_HandSoldering, symbol FB
- P3: value CONN_01X04 -> CONN_01X05; symbol CONN_01X04 -> CONN_01X05
- renumbered FB7 to FB8, FB8 to FB9
Connections:
- wire segments 177 -> 140
Other:
- note added: "PTT\nPHONE-R\nPHONE-L\nGND\nMIC"
- note removed: "PHONE-R\nPHONE-L\nGND\nMIC"
- moved on the sheet: C1, C18, C20, C6, C7, FB2, FB3, FB5, FB6, R3

Commit message: Add files via upload
Parts:
- removed FB7: FB, HERMESLITE:C_0603_HandSoldering, symbol FB
- added J1: SJ-43514-SMT, HERMESLITE:SJ-43514-SMT, symbol SJ-43514-SMT
- P1: value CONN_01X02 -> CONN_01X03; symbol CONN_01X02 -> CONN_01X03
- renumbered FB8 to FB7, FB9 to FB8, J1 to J2
Connections:
- wire segments 140 -> 183
Other:
- note added: "MIC\nPTT\nGND\n"
- note added: "PHONE-L\nPHONE-R\nGND\n"
- note removed: "DNI"
- note removed: "PTT (PHONE-L)\nPHONE\nGND\nMIC"
- moved on the sheet: C1, C10, C11, C12, C13, C14, C15, C16, C17, C18, C19, C2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

Commit message: Add files via upload
Parts:
- P1: footprint HERMESLITE:Pin_Header_Straight_1x02_Pitch2.54mm -> HERMESLITE:Pin_Header_Straight_1x03_Pitch2.54mm
- P3: footprint HERMESLITE:Pin_Header_Straight_1x04_Pitch2.54mm -> HERMESLITE:Pin_Header_Straight_1x05_Pitch2.54mm
Changed lines of the file:
@@
 F 0 "P1" V 5000 6245 50  0000 C CNN
 F 1 "CONN_01X03" V 4975 6245 50  0001 C CNN
-F 2 "HERMESLITE:Pin_Header_Straight_1x02_Pitch2.54mm" H 4875 6245 50  0001 C CNN
+F 2 "HERMESLITE:Pin_Header_Straight_1x03_Pitch2.54mm" H 4875 6245 50  0001 C CNN
 F 3 "" H 4875 6245 50  0000 C CNN
 	1    4875 6245
@@
 F 0 "P3" H 9690 3705 50  0000 C CNN
 F 1 "CONN_01X05" V 9795 3420 50  0001 C CNN
-F 2 "HERMESLITE:Pin_Header_Straight_1x04_Pitch2.54mm" H 9695 3420 50  0001 C CNN
+F 2 "HERMESLITE:Pin_Header_Straight_1x05_Pitch2.54mm" H 9695 3420 50  0001 C CNN
 F 3 "" H 9695 3420 50  0000 C CNN
 	1    9695 3420
@@
 Connection ~ 6325 4795
 Wire Wire Line
-	6200 4795 6325 4795
-Wire Wire Line
-	6325 4795 6625 4795
+	6200 4795 6625 4795
 Wire Wire Line
 	6200 4645 6200 4795
@@
 	5075 6020 5550 6020
 Wire Wire Line
-	5075 5345 5075 5845
-Wire Wire Line
-	5075 5845 5075 6020
-Wire Wire Line
-	5075 6020 5075 6720
+	5075 5345 5075 6720
 Wire Wire Line
 	9495 3520 9270 3520
 Wire Wire Line
-	8325 3620 8640 3620
-Wire Wire Line
-	8640 3620 9495 3620
+	8325 3620 9495 3620
 Wire Wire Line
 	9270 3520 9270 3695
 Connection ~ 3125 7045
 Wire Wire Line
-	3125 7020 3125 7045
-Wire Wire Line
-	3125 7045 3125 7070
+	3125 7020 3125 7070
 Wire Wire Line
 	3350 7045 3125 7045
@@
 Connection ~ 3125 6720
 Wire Wire Line
-	3125 6670 3125 6720
-Wire Wire Line
-	3125 6720 3125 6820
-Wire Wire Line
-	2885 6720 3125 6720
-Wire Wire Line
-	3125 6720 3400 6720
+	3125 6670 3125 6820
+Wire Wire Line
+	2885 6720 3400 6720
 Wire Wire Line
 	7065 4770 7065 6345
@@
 	7175 6245 7175 4970
 Wire Wire Line
-	8325 4970 8750 4970
-Wire Wire Line
-	8750 4970 8950 4970
-Wire Wire Line
-	8850 5070 8850 5170
-Wire Wire Line
-	8850 5170 8850 5270
+	8325 4970 8950 4970
+Wire Wire Line
+	8850 5070 8850 5270
 Wire Wire Line
 	8850 5070 8950 5070
 Wire Wire Line
-	4250 5670 4325 5670
-Wire Wire Line
-	4325 5670 4480 5670
-Wire Wire Line
-	4480 5670 4775 5670
+	4250 5670 4775 5670
 Wire Wire Line
 	5075 6720 4200 6720
@@
 	6625 5470 6625 5520
 Wire Wire Line
-	6325 5500 6325 5520
-Wire Wire Line
-	6325 5520 6325 5570
-Wire Wire Line
-	6325 4745 6325 4795
-Wire Wire Line
-	6325 4795 6325 5175
-Wire Wire Line
-	6325 5175 6325 5200
+	6325 5500 6325 5570
+Wire Wire Line
+	6325 4745 6325 5200
 Wire Wire Line
 	4675 2305 1875 2305
@@
 Connection ~ 3825 5670
 Wire Wire Line
-	3310 5670 3455 5670
-Wire Wire Line
-	3455 5670 3825 5670
-Wire Wire Line
-	3825 5670 3950 5670
+	3310 5670 3950 5670
 Connection ~ 7450 4770
 Connection ~ 7650 4970
 Wire Wire Line
-	7065 4770 7450 4770
-Wire Wire Line
-	7450 4770 8025 4770
+	7065 4770 8025 4770
 Wire Wire Line
 	4675 2305 4675 3845
@@
 Connection ~ 4125 4945
 Wire Wire Line
-	3455 4945 3825 4945
-Wire Wire Line
-	3825 4945 4125 4945
-Wire Wire Line
-	4125 4945 4275 4945
+	3455 4945 4275 4945
 Wire Wire Line
 	7650 5045 7650 4970
@@
 	5750 5670 5850 5670
 Wire Wire Line
-	5850 4945 5850 5670
-Wire Wire Line
-	5850 5670 5850 5845
-Wire Wire Line
-	5850 5845 5850 6020
-Wire Wire Line
-	5850 6020 5850 6080
+	5850 4945 5850 6080
 Wire Wire Line
 	5775 4945 5850 4945
@@
 Connection ~ 6050 4545
 Wire Wire Line
-	5775 4545 6050 4545
-Wire Wire Line
-	6050 4545 6325 4545
-Wire Wire Line
-	6325 4545 6625 4545
-Wire Wire Line
-	6625 4545 6850 4545
+	5775 4545 6850 4545
 Wire Wire Line
 	4875 6045 4875 5345
@@
 Connection ~ 6315 3620
 Wire Wire Line
-	6315 3420 6315 3620
-Wire Wire Line
-	6315 3620 6315 3670
+	6315 3420 6315 3670
 Wire Wire Line
 	6215 3420 6315 3420
 Wire Wire Line
-	7175 4970 7650 4970
-Wire Wire Line
-	7650 4970 8025 4970
-Wire Wire Line
-	6165 3620 6315 3620
-Wire Wire Line
-	6315 3620 8025 3620
+	7175 4970 8025 4970
+Wire Wire Line
+	6165 3620 8025 3620
 Wire Wire Line
 	1875 2205 8025 2205
@@
 	990  2305 990  1410
 Wire Wire Line
-	1175 1710 3830 1710
-Wire Wire Line
-	3830 1710 3945 1710
+	1175 1710 3945 1710
 Wire Wire Line
 	1175 2205 1175 1710
 Wire Wire Line
-	990  1410 6075 1410
-Wire Wire Line
-	6075 1410 6210 1410
+	990  1410 6210 1410
 Wire Wire Line
 	1375 6345 1300 6345
@@
 	6510 1210 9495 1210
 Wire Wire Line
-	830  3295 990  3295
-Wire Wire Line
-	990  3295 1375 3295
-Wire Wire Line
-	1375 3295 1875 3295
+	830  3295 1875 3295
 Wire Wire Line
 	990  3010 990  3295
@@
 Connection ~ 8750 4970
 Wire Wire Line
-	8325 4770 8850 4770
-Wire Wire Line
-	8850 4770 8950 4770
+	8325 4770 8950 4770
 Wire Wire Line
 	9495 1110 9345 1110
 Wire Wire Line
-	9345 1110 9345 1310
-Wire Wire Line
-	9345 1310 9345 1390
+	9345 1110 9345 1390
 Connection ~ 9345 1310
 Wire Wire Line
@@
 Connection ~ 4675 5490
 Wire Wire Line
-	3455 4945 3455 5160
-Wire Wire Line
-	3455 5160 3455 5240
+	3455 4945 3455 5240
 Wire Wire Line
 	3455 5540 3455 5670
@@
 	8640 2005 8950 2005
 Wire Wire Line
-	8325 2205 8745 2205
-Wire Wire Line
-	8745 2205 8950 2205
+	8325 2205 8950 2205
 Wire Wire Line
 	8950 5170 8850 5170
@@
 $EndComp
 Wire Wire Line
-	8850 2305 8850 2405
-Wire Wire Line
-	8850 2405 8850 2505
+	8850 2305 8850 2505
 Wire Wire Line
 	8850 2305 8950 2305

Commit message: Add files via upload
Converted to KiCad V5.0.2.
Parts:
- C1, C10, C12, C13, C14, C15, C16, C18, C19, C2, C20, C21, C4, C5, C7, C8, C9: symbol C_Small -> hermeslite-rescue:C_Small
- C11, C17, C3, C6: symbol CP_Small -> hermeslite-rescue:CP_Small
- CN1: symbol CONN_02X10 -> hermeslite-rescue:CONN_02X10
- CN12: symbol CONN_02X03 -> hermeslite-rescue:CONN_02X03
- FB1, FB2, FB3, FB4, FB5, FB6, FB7, FB8: symbol FB -> hermeslite-rescue:FB
- J1, J2: symbol SJ-43514-SMT -> hermeslite-rescue:SJ-43514-SMT
- P1: symbol CONN_01X03 -> hermeslite-rescue:CONN_01X03
- P2: symbol CONN_01X04 -> hermeslite-rescue:CONN_01X04
- P3: symbol CONN_01X05 -> hermeslite-rescue:CONN_01X05
- Q1, Q2: symbol Q_NMOS_GDS -> hermeslite-rescue:Q_NMOS_GDS
- R1, R2, R3, R4, R5: symbol R -> hermeslite-rescue:R
- U1: symbol LP2985 -> hermeslite-rescue:LP2985
- U2: symbol AK4951AEN -> hermeslite-rescue:AK4951AEN

Commit message: Add files via upload
Parts:
- removed J2: SJ-43514-SMT, HERMESLITE:SJ-43514-SMT, symbol hermeslite-rescue:SJ-43514-SMT
- added J2: PHONES, HERMESLITE:STEREO, symbol hermeslite-rescue:STEREO-hermeslite
- C1, C10, C12, C13, C14, C15, C16, C18, C19, C2, C20, C21, C4, C5, C7, C8, C9, FB1, FB2, FB3, FB4, FB5, FB6, FB7, FB8, R1, R2, R3, R4, R5: footprint HERMESLITE:C_0603_HandSoldering -> HERMESLITE:SMD-0603
- C11, C17, C3, C6: footprint HERMESLITE:TantalC_SizeB_EIA-3528_Wave -> HERMESLITE:SMD-1206
- CN1: footprint HERMESLITE:IO -> HERMESLITE:10x2
- CN12: footprint (none) -> HERMESLITE:3x2
- J1: value SJ-43514-SMT -> MIC; footprint HERMESLITE:SJ-43514-SMT -> HERMESLITE:STEREO; symbol hermeslite-rescue:SJ-43514-SMT -> hermeslite-rescue:STEREO-hermeslite
- P1: value CONN_01X03 -> CONN_01X02; footprint HERMESLITE:Pin_Header_Straight_1x03_Pitch2.54mm -> HERMESLITE:2x1; symbol hermeslite-rescue:CONN_01X03 -> hermeslite-rescue:CONN_01X02-hermeslite_HL2
- P2: footprint HERMESLITE:Pin_Header_Straight_1x04_Pitch2.54mm -> HERMESLITE:4x1
- P3: footprint HERMESLITE:Pin_Header_Straight_1x05_Pitch2.54mm -> HERMESLITE:5x1
- Q1, Q2: footprint (none) -> HERMESLITE:SOT23_2N7002
Connections:
- net GND: now also P3.3 (P3), J2.1; no longer J1.4, P1.3 (P3), P3.4 (P4)
- net at J1.2, P3.5 (P5): now also FB5.1; no longer FB6.2
- net at FB8.2: now also P3.1 (P1), J2.3; no longer P3.2 (P2)
- net at FB7.1: now also P3.2 (P2), J2.2; no longer P3.3 (P3)
- new net: FB6.2, J1.3, P3.4 (P4)
- no-connect marks 14 -> 18
Other:
- note added: "PHONE-L\n\n\nPHONE-R\nGND\n"
- note added: "PTT\nMIC\nGND\nPHONE-L\nPHONE-R"
- note added: "PTT\n\n\nMIC\nGND\n"
- note removed: "MIC\nPTT\nGND\n"
- note removed: "PHONE-L\nPHONE-R\nGND\n"
- note removed: "PTT\nPHONE-R\nPHONE-L\nGND\nMIC"
- moved on the sheet: C19, C21, FB8, P3, R4
