File: hermeslite.kicad_pcb (KiCad board)
At the start: 4 copper layers, 22.6 x 64 mm, 45 parts, among them CN1 IO20, CN12 CONN_02X03, J1 MIC, J2 PHONES, P1 CONN_01X02, P2 CONN_01X04, P3 CONN_01X05, Q1 2N7002, Q2 2N7002, U1 TPS730, U2 AK4951AEN

Commit message: Add files via upload
Parts:
- moved FB6 2.29 mm to (89.4, 126.4)
Routing:
- net Net-(C18-Pad2): track 47.7 -> 45.4 mm
- net Net-(FB6-Pad2): track 17.3 -> 17.9 mm
- net GND: vias 98 -> 97
Changed lines of the file:
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@@
     (thickness 1.6)
     (drawings 18)
-    (tracks 382)
+    (tracks 378)
     (zones 0)
     (modules 45)
@@
   )
   (module HERMESLITE:SMD-0603 (layer F.Cu)
-    (at 89.408 128.651 180)
+    (at 89.408 126.365 180)
     (attr smd)
     (fp_text reference FB6 (at 0 -1.778 270 unlocked) (layer F.SilkS)
@@
   (via (at 88.392 125.222) (size 0.6) (drill 0.3) (layers F.Cu B.Cu) (net 1))
   (via (at 90.678 125.222) (size 0.6) (drill 0.3) (layers F.Cu B.Cu) (net 1))
-  (via (at 88.392 127.508) (size 0.6) (drill 0.3) (layers F.Cu B.Cu) (net 1))
-  (via (at 90.678 127.508) (size 0.6) (drill 0.3) (layers F.Cu B.Cu) (net 1))
+  (via (at 90.678 127.762) (size 0.6) (drill 0.3) (layers F.Cu B.Cu) (net 1))
   (via (at 86.106 127.508) (size 0.6) (drill 0.3) (layers F.Cu B.Cu) (net 1))
-  (via (at 86.106 129.794) (size 0.6) (drill 0.3) (layers F.Cu B.Cu) (net 1))
-  (via (at 86.106 132.334) (size 0.6) (drill 0.3) (layers F.Cu B.Cu) (net 1))
   (via (at 86.106 134.366) (size 0.6) (drill 0.3) (layers F.Cu B.Cu) (net 1))
   (via (at 76.708 134.366) (size 0.6) (drill 0.3) (layers F.Cu B.Cu) (net 1))
   (via (at 76.708 132.08) (size 0.6) (drill 0.3) (layers F.Cu B.Cu) (net 1))
-  (via (at 74.422 131.064) (size 0.6) (drill 0.3) (layers F.Cu B.Cu) (net 1))
+  (via (at 74.676 131.064) (size 0.6) (drill 0.3) (layers F.Cu B.Cu) (net 1))
   (via (at 71.882 131.064) (size 0.6) (drill 0.3) (layers F.Cu B.Cu) (net 1))
   (via (at 71.882 128.524) (size 0.6) (drill 0.3) (layers F.Cu B.Cu) (net 1))
   (via (at 71.882 125.984) (size 0.6) (drill 0.3) (layers F.Cu B.Cu) (net 1))
-  (via (at 74.422 125.984) (size 0.6) (drill 0.3) (layers F.Cu B.Cu) (net 1))
+  (via (at 74.676 125.984) (size 0.6) (drill 0.3) (layers F.Cu B.Cu) (net 1))
   (via (at 71.882 121.412) (size 0.6) (drill 0.3) (layers F.Cu B.Cu) (net 1))
-  (via (at 74.422 121.412) (size 0.6) (drill 0.3) (layers F.Cu B.Cu) (net 1))
+  (via (at 74.676 121.412) (size 0.6) (drill 0.3) (layers F.Cu B.Cu) (net 1))
   (via (at 78.994 121.412) (size 0.6) (drill 0.3) (layers F.Cu B.Cu) (net 1))
   (via (at 83.82 121.412) (size 0.6) (drill 0.3) (layers F.Cu B.Cu) (net 1))
@@
   (via (at 77.216 118.872) (size 0.6) (drill 0.3) (layers F.Cu B.Cu) (net 1))
   (via (at 71.882 117.602) (size 0.6) (drill 0.3) (layers F.Cu B.Cu) (net 1))
-  (via (at 74.676 117.602) (size 0.6) (drill 0.3) (layers F.Cu B.Cu) (net 1))
+  (via (at 75.692 117.602) (size 0.6) (drill 0.3) (layers F.Cu B.Cu) (net 1))
   (via (at 71.882 114.808) (size 0.6) (drill 0.3) (layers F.Cu B.Cu) (net 1))
-  (via (at 74.676 114.808) (size 0.6) (drill 0.3) (layers F.Cu B.Cu) (net 1))
+  (via (at 75.692 114.808) (size 0.6) (drill 0.3) (layers F.Cu B.Cu) (net 1))
   (via (at 82.042 114.808) (size 0.6) (drill 0.3) (layers F.Cu B.Cu) (net 1))
   (via (at 78.232 114.808) (size 0.6) (drill 0.3) (layers F.Cu B.Cu) (net 1))
@@
   (via (at 80.772 112.014) (size 0.6) (drill 0.3) (layers F.Cu B.Cu) (net 1))
   (via (at 71.882 111.252) (size 0.6) (drill 0.3) (layers F.Cu B.Cu) (net 1))
-  (via (at 74.676 111.252) (size 0.6) (drill 0.3) (layers F.Cu B.Cu) (net 1))
+  (via (at 75.692 111.252) (size 0.6) (drill 0.3) (layers F.Cu B.Cu) (net 1))
   (via (at 71.882 108.204) (size 0.6) (drill 0.3) (layers F.Cu B.Cu) (net 1))
   (via (at 71.882 105.41) (size 0.6) (drill 0.3) (layers F.Cu B.Cu) (net 1))
-  (via (at 74.676 105.41) (size 0.6) (drill 0.3) (layers F.Cu B.Cu) (net 1))
+  (via (at 75.692 105.41) (size 0.6) (drill 0.3) (layers F.Cu B.Cu) (net 1))
   (via (at 71.882 101.854) (size 0.6) (drill 0.3) (layers F.Cu B.Cu) (net 1))
   (via (at 71.882 99.06) (size 0.6) (drill 0.3) (layers F.Cu B.Cu) (net 1))
@@
   (via (at 78.994 87.884) (size 0.6) (drill 0.3) (layers F.Cu B.Cu) (net 1))
   (via (at 78.994 84.582) (size 0.6) (drill 0.3) (layers F.Cu B.Cu) (net 1))
-  (via (at 89.154 132.08) (size 5.3) (drill 3.3) (layers F.Cu B.Cu) (net 1))
+  (via (at 89.154 131.96) (size 6.3) (drill 3.3) (layers F.Cu B.Cu) (net 1))
+  (via (at 86.106 130.048) (size 0.6) (drill 0.3) (layers F.Cu B.Cu) (net 1))
+  (via (at 88.392 127.762) (size 0.6) (drill 0.3) (layers F.Cu B.Cu) (net 1))
   (via (at 89.154 103.886) (size 0.6) (drill 0.3) (layers F.Cu B.Cu) (net 2))
   (segment (start 74.041 99.221) (end 74.04 99.22) (width 0.6096) (layer B.Cu) (net 2))
@@
   (segment (start 91.44 94.488) (end 85.598 94.488) (width 0.254) (layer F.Cu) (net 15))
   (segment (start 92.202 95.25) (end 91.44 94.488) (width 0.254) (layer F.Cu) (net 15))
-  (segment (start 92.202 127.762) (end 92.202 95.25) (width 0.254) (layer F.Cu) (net 15))
-  (segment (start 90.17 128.651) (end 91.313 128.651) (width 0.254) (layer F.Cu) (net 15))
-  (segment (start 91.313 128.651) (end 92.202 127.762) (width 0.254) (layer F.Cu) (net 15))
+  (segment (start 90.17 126.365) (end 91.313 126.365) (width 0.254) (layer F.Cu) (net 15))
+  (segment (start 91.313 126.365) (end 92.202 125.476) (width 0.254) (layer F.Cu) (net 15))
+  (segment (start 92.202 125.476) (end 92.202 95.25) (width 0.254) (layer F.Cu) (net 15))
   (via (at 85.344 102.444938) (size 0.6) (drill 0.3) (layers F.Cu B.Cu) (net 16))
   (segment (start 86.185714 113.478732) (end 86.272857 113.391589) (width 0.254) (layer F.Cu) (net 16))
@@
   (segment (start 79.5 123.4) (end 80.982 123.4) (width 0.254) (layer F.Cu) (net 36))
   (segment (start 80.982 123.4) (end 81.788 124.206) (width 0.254) (layer F.Cu) (net 36))
-  (segment (start 87.503 128.651) (end 88.646 128.651) (width 0.254) (layer F.Cu) (net 36))
-  (segment (start 86.723001 129.430999) (end 87.503 128.651) (width 0.254) (layer F.Cu) (net 36))
-  (segment (start 86.723001 130.192999) (end 86.723001 129.430999) (width 0.254) (layer F.Cu) (net 36))
-  (segment (start 84.074 131.064) (end 85.852 131.064) (width 0.254) (layer F.Cu) (net 36))
-  (segment (start 85.852 131.064) (end 86.723001 130.192999) (width 0.254) (layer F.Cu) (net 36))
+  (segment (start 88.646 126.492) (end 88.646 126.365) (width 0.254) (layer F.Cu) (net 36))
+  (segment (start 84.074 131.064) (end 88.646 126.492) (width 0.254) (layer F.Cu) (net 36))
   (segment (start 76.708 130.608) (end 79.5 133.4) (width 0.254) (layer F.Cu) (net 38))
   (segment (start 76.708 120.396) (end 76.708 130.608) (width 0.254) (layer F.Cu) (net 38))
