File: hermeslite.kicad_pcb (KiCad board)
At the start: 4 copper layers, 22.6 x 64 mm, 45 parts, among them CN1 IO20, CN12 CONN_02X03, J1 MIC, J2 PHONES, P1 CONN_01X02, P2 CONN_01X04, P3 CONN_01X05, Q1 2N7002, Q2 2N7002, U1 TPS730, U2 AK4951AEN

Commit message: Add files via upload
Parts:
- moved FB6 2.67 mm to (86.7, 126.4), turned to 270 degrees
- moved C5 0.06 mm to (91.2, 105.7)
Routing:
- net Net-(C18-Pad2): track 45.4 -> 47.8 mm
- net Net-(FB6-Pad2): track 17.9 -> 16.4 mm
- net Net-(FB7-Pad1): track 20.0 -> 19.5 mm
- net Net-(P1-Pad1): track 11.0 -> 10.5 mm
- net GND: vias 97 -> 95
